File: EN022-001_cpu-power-base/vselect.kicad_sch (KiCad schematic)
At the start: 5 parts, among them U1 TPS2113PW

Commit message: applied page layout
Other:
- title: (none) -> Power supply section
Changed lines of the file:
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@@
 	(generator_version "8.0")
 	(paper "A4")
+	(title_block
+		(title "Power supply section")
+		(date "2024-09-19")
+		(rev "A")
+	)
 	(junction
 		(at 36.83 26.67)

Commit message: first cimplete  version of CPU POWER BASE
Parts:
- renumbered C2 to C5, C3 to C8, C4 to C9, R2 to R11, U1 to U2
